Commit message: refine collision group filter

File: assets/linker_hand/L25_dof_urdf.urdf (robot description, URDF)
Before this commit: robot L25-dof-urdf, 22 links, 21 joints
Links:
- link base_link: geometry collision mesh filename=meshes/base_link.STL; visual mesh filename=meshes/base_link.STL
- link thumb_joint1: geometry collision mesh filename=meshes/thumb_joint1.STL; visual mesh filename=meshes/thumb_joint1.STL
- link thumb_joint2: geometry collision mesh filename=meshes/thumb_joint2.STL; visual mesh filename=meshes/thumb_joint2.STL

Commit message: TA Optuna初步训练成功

File: assets/linker_hand/L25_dof_urdf.urdf (robot description, URDF)
Before this commit: robot L25-dof-urdf, 22 links, 21 joints
Links:
- link base_link: geometry visual mesh filename=meshes/base_link.STL
